Commit message: okish,nav working,tf fixed

File: ros_ws/src/lampo_description/urdf/sweepee/sweepee_omni.xacro (robot description, xacro)
@@ -54,226 +54,212 @@
       <child link="${prefix}front_laser" /> -->
     </joint>
-      <link name="${prefix}rear_laser" />
-    <joint name="${prefix}rear_laser_joint" type="fixed">
-      <origin xyz="${-base_x_size/2+0.15} 0.0 ${base_z_size/2+0.085}" rpy="0 0 ${M_PI}" />
-      <parent link="${prefix}base_link_sweepee" />
-      <child link="${prefix}rear_laser" />
-    </joint>
-      <link name='${prefix}front_left_wheel'>
-        <inertial>
-          <mass value="5"/>
-          <inertia ixx="0.145"  ixy="0"  ixz="0" iyy="0.145" iyz="0" izz="0.125" />
-        </inertial>
-        <visual>
-          <geometry>
-            <cylinder length="0.05" radius="0.1"/>
-          </geometry>
-        </visual>
-        <collision>
-          <geometry>
-            <cylinder length="0.05" radius="0.1"/>
-          </geometry>
-        </collision>
-      </link>
-      <link name='${prefix}rear_left_wheel'>
-        <inertial>
-          <mass value="5"/>
-          <inertia ixx="0.145"  ixy="0"  ixz="0" iyy="0.145" iyz="0" izz="0.125" />
-        </inertial>
-        <visual>
-          <geometry>
-            <cylinder length="0.05" radius="0.1"/>
-          </geometry>
-        </visual>
-        <collision>
-          <geometry>
-            <cylinder length="0.05" radius="0.1"/>
-          </geometry>
-        </collision>
-      </link>
-      <link name='${prefix}front_right_wheel'>
-        <inertial>
-          <mass value="5"/>
-          <inertia ixx="0.145"  ixy="0"  ixz="0" iyy="0.145" iyz="0" izz="0.125" />
-        </inertial>
-        <visual>
-          <geometry>
-            <cylinder length="0.05" radius="0.1"/>
-          </geometry>
-        </visual>
-        <collision>
-          <geometry>
-            <cylinder length="0.05" radius="0.1"/>
-          </geometry>
-        </collision>
-      </link>
-      <link name='${prefix}rear_right_wheel'>
-        <inertial>
-          <mass value="5"/>
-          <inertia ixx="0.145"  ixy="0"  ixz="0" iyy="0.145" iyz="0" izz="0.125" />
-        </inertial>
-        <visual>
-          <geometry>
-            <cylinder length="0.05" radius="0.1"/>
-          </geometry>
-        </visual>
-        <collision>
-          <geometry>
-            <cylinder length="0.05" radius="0.1"/>
-          </geometry>
-        </collision>
-      </link>
-      <!-- <gazebo reference="${prefix}front_left_wheel">
-        <mu1>0.5</mu1>
-        <mu2>0.1</mu2>
-        <fdir1 gz:expressed_in='${prefix}base_footprint'>1 -1 0</fdir1>
-      </gazebo>
-      <gazebo reference="${prefix}rear_left_wheel">
-        <mu1>0.0</mu1>
-        <mu2>0.0</mu2>
-        <fdir1 gz:expressed_in='${prefix}base_footprint'>1 1 0</fdir1>
-      </gazebo>
-      <gazebo reference="${prefix}front_right_wheel">
-        <mu1>0.5</mu1>
-        <mu2>0.1</mu2>
-        <fdir1 gz:expressed_in='${prefix}base_footprint'>1 1 0</fdir1>
-      </gazebo>
-      <gazebo reference="${prefix}rear_right_wheel">
-        <mu1>0.0</mu1>
-        <mu2>0.0</mu2>
-        <fdir1 gz:expressed_in='${prefix}base_footprint'>1 -1 0</fdir1>
-      </gazebo> -->
-      <gazebo reference='${prefix}front_left_wheel'>
-        <collision>
-          <surface>
-            <friction>
-              <ode>
-                <mu>1.0</mu>
-                <mu2>0.0</mu2>
-                <fdir1 gz:expressed_in="${prefix}base_footprint">1 -1 0</fdir1>
-              </ode>
-            </friction>
-          </surface>
-        </collision>
-      </gazebo>
-      <gazebo reference='${prefix}front_right_wheel'>
-        <collision>
-          <surface>
-            <friction>
-              <ode>
-                <mu>1.0</mu>
-                <mu2>0.0</mu2>
-                <fdir1 gz:expressed_in="${prefix}base_footprint">1 1 0</fdir1>
-              </ode>
-            </friction>
-          </surface>
-        </collision>
-      </gazebo>
-      <gazebo reference='${prefix}rear_left_wheel'>
-        <collision>
-          <surface>
-            <friction>
-              <ode>
-                <mu>1.0</mu>
-                <mu2>0.0</mu2>
-                <fdir1 gz:expressed_in="${prefix}base_footprint">1 1 0</fdir1>
-              </ode>
-            </friction>
-          </surface>
-        </collision>
-      </gazebo>
-      <gazebo reference='${prefix}rear_right_wheel'>
-        <collision>
-          <surface>
-            <friction>
-              <ode>
-                <mu>1.0</mu>
-                <mu2>0.0</mu2>
-                <fdir1 gz:expressed_in="${prefix}base_footprint">1 -1 0</fdir1>
-              </ode>
-            </friction>
-          </surface>
-        </collision>
-      </gazebo>
-      <joint name='${prefix}front_left_wheel_joint' type='revolute'>
-        <origin xyz="0.3 0.25 0.1" rpy="-1.5707 0 0"/>
-        <parent link="${prefix}base_link_sweepee"/>
-        <child link="${prefix}front_left_wheel"/>
-        <axis xyz="0 0 1"/>
-        <limit effort="10000.0" lower="-1.79769e+308" upper="1.79769e+308" velocity="15.1"/>
-      </joint>
-      <joint name='${prefix}front_right_wheel_joint' type='revolute'>
-        <origin xyz="0.3 -0.25 0.1" rpy="-1.5707 0 0"/>
-        <parent link="${prefix}base_link_sweepee"/>
-        <child link="${prefix}front_right_wheel"/>
-        <axis xyz="0 0 1"/>
-        <limit effort="10000.0" lower="-1.79769e+308" upper="1.79769e+308" velocity="15.1"/>
-      </joint>
-      <joint name='${prefix}rear_left_wheel_joint' type='revolute'>
-        <origin xyz="-0.3 0.25 0.1" rpy="-1.5707 0 0"/>
-        <parent link="${prefix}base_link_sweepee"/>
-        <child link="${prefix}rear_left_wheel"/>
-        <axis xyz="0 0 1"/>
-        <limit effort="10000.0" lower="-1.79769e+308" upper="1.79769e+308" velocity="15.1"/>
-      </joint>
-      <joint name='${prefix}rear_right_wheel_joint' type='revolute'>
-        <origin xyz="-0.3 -0.25 0.1" rpy="-1.5707 0 0"/>
-        <parent link="${prefix}base_link_sweepee"/>
-        <child link="${prefix}rear_right_wheel"/>
-        <axis xyz="0 0 1"/>
-        <limit effort="10000.0" lower="-1.79769e+308" upper="1.79769e+308" velocity="15.1"/>
-      </joint>
-  <gazebo reference="${prefix}front_laser">
-    <sensor name='gpu_lidar' type='gpu_lidar'>
-        <pose relative_to='${prefix}front_laser'>0 0 0 0 0 0</pose>
-        <gz_frame_id>${prefix}front_laser</gz_frame_id>
-        <topic>${prefix}lidar</topic>
-        <update_rate>10</update_rate>
-        <lidar>
-            <scan>
-                <horizontal>
-                    <samples>640</samples>
-                    <resolution>1</resolution>
-                    <min_angle>-1.396263</min_angle>
-                    <max_angle>1.396263</max_angle>
-                </horizontal>
-                <vertical>
-                    <samples>1</samples>
-                    <resolution>0.01</resolution>
-                    <min_angle>0</min_angle>
-                    <max_angle>0</max_angle>
-                </vertical>
-            </scan>
-            <range>
-                <min>0.15</min>
-                <max>30.0</max>
-                <resolution>0.01</resolution>
-            </range>
-        </lidar>
-        <always_on>1</always_on>
-        <visualize>true</visualize>
-    </sensor>
-  </gazebo>
-  <gazebo>
-    <plugin
-      filename="gz-sim-mecanum-drive-system"
-      name="gz::sim::systems::MecanumDrive">
-      <front_left_joint>${prefix}front_left_wheel_joint</front_left_joint>
-      <front_right_joint>${prefix}front_right_wheel_joint</front_right_joint>
-      <back_left_joint>${prefix}rear_left_wheel_joint</back_left_joint>
-      <back_right_joint>${prefix}rear_right_wheel_joint</back_right_joint>
-      <wheel_separation>0.5</wheel_separation>
-      <wheelbase>0.6</wheelbase>
-      <wheel_radius>0.1</wheel_radius>
-      <min_acceleration>-5</min_acceleration>
-      <max_acceleration>5</max_acceleration>
-      <max_velocity>1.5</max_velocity>
-      <topic>${prefix}cmd_vel</topic>
-      <frame_id>${prefix}odom</frame_id>
-      <odom_topic>${prefix}odom</odom_topic>
-      <child_frame_id>${prefix}base_footprint</child_frame_id>
-      <tf_topic>tf</tf_topic>
-    </plugin>
-  </gazebo>
+    <gazebo reference='${prefix}front_laser_joint'>
+      <disableFixedJointLumping>true</disableFixedJointLumping>
+      <preserveFixedJoint>true</preserveFixedJoint>
+    </gazebo>
+    <link name='${prefix}front_left_wheel'>
+      <inertial>
+        <mass value="5"/>
+        <inertia ixx="0.145"  ixy="0"  ixz="0" iyy="0.145" iyz="0" izz="0.125" />
+      </inertial>
+      <visual>
+        <geometry>
+          <cylinder length="0.05" radius="0.1"/>
+        </geometry>
+      </visual>
+      <collision>
+        <geometry>
+          <cylinder length="0.05" radius="0.1"/>
+        </geometry>
+      </collision>
+    </link>
+    <link name='${prefix}rear_left_wheel'>
+      <inertial>
+        <mass value="5"/>
+        <inertia ixx="0.145"  ixy="0"  ixz="0" iyy="0.145" iyz="0" izz="0.125" />
+      </inertial>
+      <visual>
+        <geometry>
+          <cylinder length="0.05" radius="0.1"/>
+        </geometry>
+      </visual>
+      <collision>
+        <geometry>
+          <cylinder length="0.05" radius="0.1"/>
+        </geometry>
+      </collision>
+    </link>
+    <link name='${prefix}front_right_wheel'>
+      <inertial>
+        <mass value="5"/>
+        <inertia ixx="0.145"  ixy="0"  ixz="0" iyy="0.145" iyz="0" izz="0.125" />
+      </inertial>
+      <visual>
+        <geometry>
+          <cylinder length="0.05" radius="0.1"/>
+        </geometry>
+      </visual>
+      <collision>
+        <geometry>
+          <cylinder length="0.05" radius="0.1"/>
+        </geometry>
+      </collision>
+    </link>
+    <link name='${prefix}rear_right_wheel'>
+      <inertial>
+        <mass value="5"/>
+        <inertia ixx="0.145"  ixy="0"  ixz="0" iyy="0.145" iyz="0" izz="0.125" />
+      </inertial>
+      <visual>
+        <geometry>
+          <cylinder length="0.05" radius="0.1"/>
+        </geometry>
+      </visual>
+      <collision>
+        <geometry>
+          <cylinder length="0.05" radius="0.1"/>
+        </geometry>
+      </collision>
+    </link>
+    <gazebo reference='${prefix}front_left_wheel'>
+      <collision>
+        <surface>
+          <friction>
+            <ode>
+              <mu>1.0</mu>
+              <mu2>0.0</mu2>
+              <fdir1 gz:expressed_in="${prefix}base_footprint">1 -1 0</fdir1>
+            </ode>
+          </friction>
+        </surface>
+      </collision>
+    </gazebo>
+    <gazebo reference='${prefix}front_right_wheel'>
+      <collision>
+        <surface>
+          <friction>
+            <ode>
+              <mu>1.0</mu>
+              <mu2>0.0</mu2>
+              <fdir1 gz:expressed_in="${prefix}base_footprint">1 1 0</fdir1>
+            </ode>
+          </friction>
+        </surface>
+      </collision>
+    </gazebo>
+    <gazebo reference='${prefix}rear_left_wheel'>
+      <collision>
+        <surface>
+          <friction>
+            <ode>
+              <mu>1.0</mu>
+              <mu2>0.0</mu2>
+              <fdir1 gz:expressed_in="${prefix}base_footprint">1 1 0</fdir1>
+            </ode>
+          </friction>
+        </surface>
+      </collision>
+    </gazebo>
+    <gazebo reference='${prefix}rear_right_wheel'>
+      <collision>
+        <surface>
+          <friction>
+            <ode>
+              <mu>1.0</mu>
+              <mu2>0.0</mu2>
+              <fdir1 gz:expressed_in="${prefix}base_footprint">1 -1 0</fdir1>
+            </ode>
+          </friction>
+        </surface>
+      </collision>
+    </gazebo>
+    <joint name='${prefix}front_left_wheel_joint' type='revolute'>
+      <origin xyz="0.3 0.25 0.1" rpy="-1.5707 0 0"/>
+      <parent link="${prefix}base_link_sweepee"/>
+      <child link="${prefix}front_left_wheel"/>
+      <axis xyz="0 0 1"/>
+      <limit effort="10000.0" lower="-1.79769e+308" upper="1.79769e+308" velocity="15.1"/>
+    </joint>
+    <joint name='${prefix}front_right_wheel_joint' type='revolute'>
+      <origin xyz="0.3 -0.25 0.1" rpy="-1.5707 0 0"/>
+      <parent link="${prefix}base_link_sweepee"/>
+      <child link="${prefix}front_right_wheel"/>
+      <axis xyz="0 0 1"/>
+      <limit effort="10000.0" lower="-1.79769e+308" upper="1.79769e+308" velocity="15.1"/>
+    </joint>
+    <joint name='${prefix}rear_left_wheel_joint' type='revolute'>
+      <origin xyz="-0.3 0.25 0.1" rpy="-1.5707 0 0"/>
+      <parent link="${prefix}base_link_sweepee"/>
+      <child link="${prefix}rear_left_wheel"/>
+      <axis xyz="0 0 1"/>
+      <limit effort="10000.0" lower="-1.79769e+308" upper="1.79769e+308" velocity="15.1"/>
+    </joint>
+    <joint name='${prefix}rear_right_wheel_joint' type='revolute'>
+      <origin xyz="-0.3 -0.25 0.1" rpy="-1.5707 0 0"/>
+      <parent link="${prefix}base_link_sweepee"/>
+      <child link="${prefix}rear_right_wheel"/>
+      <axis xyz="0 0 1"/>
+      <limit effort="10000.0" lower="-1.79769e+308" upper="1.79769e+308" velocity="15.1"/>
+    </joint>
+    <gazebo reference="${prefix}base_link_sweepee">
+      <sensor name="imu_sensor" type="imu">
+          <always_on>1</always_on>
+          <update_rate>50</update_rate>
+          <visualize>true</visualize>
+          <topic>${prefix}imu</topic>
+      </sensor>
+    </gazebo>
+    <gazebo reference="${prefix}front_laser">
+      <sensor name='gpu_lidar' type='gpu_lidar'>
+          <pose relative_to='${prefix}front_laser'>0 0 0 0 0 0</pose>
+          <frame_id>${prefix}front_laser</frame_id>
+          <topic>${prefix}lidar</topic>
+          <update_rate>10</update_rate>
+          <lidar>
+              <scan>
+                  <horizontal>
+                      <samples>640</samples>
+                      <resolution>1</resolution>
+                      <min_angle>-1.396263</min_angle>
+                      <max_angle>1.396263</max_angle>
+                  </horizontal>
+                  <vertical>
+                      <samples>1</samples>
+                      <resolution>0.01</resolution>
+                      <min_angle>0</min_angle>
+                      <max_angle>0</max_angle>
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
Commit message: whole mm working with camera

File: ros_ws/src/lampo_description/urdf/sweepee/sweepee_omni.xacro (robot description, xacro)
@@ -205,5 +205,5 @@
       <sensor name="imu_sensor" type="imu">
           <always_on>1</always_on>
-          <update_rate>50</update_rate>
+          <update_rate>10</update_rate>
           <visualize>true</visualize>
           <topic>${prefix}imu</topic>

File: ros_ws/src/lampo_description/urdf/system.urdf.xacro (robot description, xacro)
@@ -2,4 +2,5 @@
 <robot name="mm1" xmlns:xacro="http://ros.org/wiki/xacro" xmlns:gz="http://gazebosim.org/schema">>
   <xacro:arg name="omni" default="false" />
+  <xacro:arg name="mm" default="false" />
   <xacro:if value="$(arg omni)">
     <xacro:include filename="$(find lampo_description)/urdf/sweepee/sweepee_omni.xacro" />
@@ -8,10 +9,122 @@
     <xacro:include filename="$(find lampo_description)/urdf/sweepee/sweepee_diff.xacro" />
   </xacro:unless>
-    <!-- Simulation parameters -->
-  <xacro:arg name="sim_gz" default="false" />
-  <xacro:arg name="simulation_controllers" default="error_default" />
-  <xacro:property name="M_PI" value="3.14159"/>
   <xacro:sweepee  prefix="$(arg prefix)">
     <origin xyz="0 0 0" rpy="0 0 0" />
   </xacro:sweepee>
+  <!-- UR -->
+  <xacro:if value="$(arg mm)">
+    <xacro:arg name="name" default="ur"/>
+    <xacro:include filename="$(find ur_description)/urdf/ur_macro.xacro"/>
+    <xacro:include filename="$(find ur_simulation_gz)/urdf/ur_gz.ros2_control.xacro" />
+    <xacro:arg name="ur_type" default="ur20"/>
+    <xacro:arg name="tf_prefix" default="sweepee_1/" />
+    <xacro:arg name="joint_limit_params" default="$(find ur_description)/config/$(arg ur_type)/joint_limits.yaml"/>
+    <xacro:arg name="kinematics_params" default="$(find ur_description)/config/$(arg ur_type)/default_kinematics.yaml"/>
+    <xacro:arg name="physical_params" default="$(find ur_description)/config/$(arg ur_type)/physical_parameters.yaml"/>
+    <xacro:arg name="visual_params" default="$(find ur_description)/config/$(arg ur_type)/visual_parameters.yaml"/>
+    <xacro:arg name="transmission_hw_interface" default=""/>
+    <xacro:arg name="safety_limits" default="false"/>
+    <xacro:arg name="safety_pos_margin" default="0.15"/>
+    <xacro:arg name="safety_k_position" default="20"/>
+    <xacro:arg name="simulation_controllers" default="$(find lampo_description)/config/ur_controllers.yaml" />
+    <xacro:arg name="ros_namespace" default="sweepee_1" />
+    <!-- arm -->
+    <xacro:ur_robot
+      name="$(arg name)"
+      tf_prefix="$(arg tf_prefix)"
+      parent="$(arg prefix)base_link_sweepee"
+      joint_limits_parameters_file="$(arg joint_limit_params)"
+      kinematics_parameters_file="$(arg kinematics_params)"
+      physical_parameters_file="$(arg physical_params)"
+      visual_parameters_file="$(arg visual_params)"
+      safety_limits="$(arg safety_limits)"
+      safety_pos_margin="$(arg safety_pos_margin)"
+      safety_k_position="$(arg safety_k_position)"
+      force_abs_paths="true"
+      >
+      <origin xyz="0 0 0.3" rpy="0 0 0" />          <!-- position robot in the world -->
+    </xacro:ur_robot>
+    <gazebo reference="world">
+    </gazebo>
+    <gazebo>
+      <plugin filename="gz_ros2_control-system" name="gz_ros2_control::GazeboSimROS2ControlPlugin">
+        <parameters>$(arg simulation_controllers)</parameters>
+        <ros>
+          <namespace>$(arg ros_namespace)</namespace>
+        </ros>
+      </plugin>
+    </gazebo>
+    <!-- ros2 control instance -->
+    <xacro:ur_ros2_control
+      name="$(arg name)"
+      tf_prefix="$(arg tf_prefix)"
+      transmission_hw_interface="$(arg transmission_hw_interface)"
+    />
+    <link name="$(arg prefix)cam_link">
+      <inertial>
+        <mass value="0.2"/>
+        <inertia ixx="0.0145"  ixy="0"  ixz="0" iyy="0.0145" iyz="0" izz="0.02125" />
+      </inertial>
+    </link>
+    <joint name="$(arg prefix)cam_joint" type="fixed">
+      <origin xyz="0.0 0.0 0.1" rpy="0 0 0" />
+      <parent link="$(arg prefix)wrist_2_link" />
+      <child link="$(arg prefix)cam_link" />
+    </joint>
+    <gazebo reference='$(arg prefix)cam_joint'>
+      <disableFixedJointLumping>true</disableFixedJointLumping>
+      <preserveFixedJoint>true</preserveFixedJoint>
+    </gazebo>
+    <gazebo reference="$(arg prefix)cam_link">
+      <sensor name="rs_front" type="rgbd_camera">
+        <pose>0.0 0.0 0.0 0.0 0.0 0.0</pose>
+        <always_on>1</always_on>
+        <update_rate>30</update_rate>
+        <topic>$(arg prefix)rgbd_camera</topic>
+        <camera name="rs_front">
+          <horizontal_fov>1.50098</horizontal_fov>
+          <lens>
+            <intrinsics>
+              <!-- fx = fy = width / ( 2 * tan (hfov / 2 ) ) -->
+              <fx>343.159</fx>
+              <fy>343.159</fy>
+              <!-- cx = ( width - 1 ) / 2 -->
+              <cx>319.5</cx>
+              <!-- cy = ( height - 1 ) / 2 -->
+              <cy>179.5</cy>
+              <s>0</s>
+            </intrinsics>
+          </lens>
+          <distortion>
+            <k1>0.0</k1>
+            <k2>0.0</k2>
+            <k3>0.0</k3>
+            <p1>0.0</p1>
+            <p2>0.0</p2>
+            <center>0.5 0.5</center>
+          </distortion>
+          <image>
+            <width>640</width>
+            <height>360</height>
+            <format>R8G8B8</format>
+          </image>
+          <clip>
+            <near>0.01</near>
+            <far>300</far>
+          </clip>
+          <depth_camera>
+            <clip>
+              <near>0.1</near>
+              <far>10</far>
+            </clip>
+          </depth_camera>
+          <noise>
+            <type>gaussian</type>
+            <mean>0</mean>
+            <stddev>0.007</stddev>
+          </noise>
+        </camera>
+      </sensor>
+    </gazebo>
+  </xacro:if>
 </robot>
