Commit message: pre dynamic names, gripper ok

File: ros_ws/src/lampo_description/urdf/system.urdf.xacro (robot description, xacro)
@@ -12,119 +12,7 @@
     <origin xyz="0 0 0" rpy="0 0 0" />
   </xacro:sweepee>
-  <!-- UR -->
+  <!-- Mobile Manipulator Configuration -->
   <xacro:if value="$(arg mm)">
-    <xacro:arg name="name" default="ur"/>
-    <xacro:include filename="$(find ur_description)/urdf/ur_macro.xacro"/>
-    <xacro:include filename="$(find ur_simulation_gz)/urdf/ur_gz.ros2_control.xacro" />
-    <xacro:arg name="ur_type" default="ur20"/>
-    <xacro:arg name="tf_prefix" default="sweepee_1/" />
-    <xacro:arg name="joint_limit_params" default="$(find ur_description)/config/$(arg ur_type)/joint_limits.yaml"/>
-    <xacro:arg name="kinematics_params" default="$(find ur_description)/config/$(arg ur_type)/default_kinematics.yaml"/>
-    <xacro:arg name="physical_params" default="$(find ur_description)/config/$(arg ur_type)/physical_parameters.yaml"/>
-    <xacro:arg name="visual_params" default="$(find ur_description)/config/$(arg ur_type)/visual_parameters.yaml"/>
-    <xacro:arg name="transmission_hw_interface" default=""/>
-    <xacro:arg name="safety_limits" default="false"/>
-    <xacro:arg name="safety_pos_margin" default="0.15"/>
-    <xacro:arg name="safety_k_position" default="20"/>
-    <xacro:arg name="simulation_controllers" default="$(find lampo_description)/config/ur_controllers.yaml" />
-    <xacro:arg name="ros_namespace" default="sweepee_1" />
-    <!-- arm -->
-    <xacro:ur_robot
-      name="$(arg name)"
-      tf_prefix="$(arg tf_prefix)"
-      parent="$(arg prefix)base_link_sweepee"
-      joint_limits_parameters_file="$(arg joint_limit_params)"
-      kinematics_parameters_file="$(arg kinematics_params)"
-      physical_parameters_file="$(arg physical_params)"
-      visual_parameters_file="$(arg visual_params)"
-      safety_limits="$(arg safety_limits)"
-      safety_pos_margin="$(arg safety_pos_margin)"
-      safety_k_position="$(arg safety_k_position)"
-      force_abs_paths="true"
-      >
-      <origin xyz="0 0 0.3" rpy="0 0 0" />          <!-- position robot in the world -->
-    </xacro:ur_robot>
-    <gazebo reference="world">
-    </gazebo>
-    <gazebo>
-      <plugin filename="gz_ros2_control-system" name="gz_ros2_control::GazeboSimROS2ControlPlugin">
-        <parameters>$(arg simulation_controllers)</parameters>
-        <ros>
-          <namespace>$(arg ros_namespace)</namespace>
-        </ros>
-      </plugin>
-    </gazebo>
-    <!-- ros2 control instance -->
-    <xacro:ur_ros2_control
-      name="$(arg name)"
-      tf_prefix="$(arg tf_prefix)"
-      transmission_hw_interface="$(arg transmission_hw_interface)"
-    />
-    <link name="$(arg prefix)cam_link">
-      <inertial>
-        <mass value="0.2"/>
-        <inertia ixx="0.0145"  ixy="0"  ixz="0" iyy="0.0145" iyz="0" izz="0.02125" />
-      </inertial>
-    </link>
-    <joint name="$(arg prefix)cam_joint" type="fixed">
-      <origin xyz="0.0 0.0 0.1" rpy="0 0 0" />
-      <parent link="$(arg prefix)wrist_2_link" />
-      <child link="$(arg prefix)cam_link" />
-    </joint>
-    <gazebo reference='$(arg prefix)cam_joint'>
-      <disableFixedJointLumping>true</disableFixedJointLumping>
-      <preserveFixedJoint>true</preserveFixedJoint>
-    </gazebo>
-    <gazebo reference="$(arg prefix)cam_link">
-      <sensor name="rs_front" type="rgbd_camera">
-        <pose>0.0 0.0 0.0 0.0 0.0 0.0</pose>
-        <always_on>1</always_on>
-        <update_rate>30</update_rate>
-        <topic>$(arg prefix)rgbd_camera</topic>
-        <camera name="rs_front">
-          <horizontal_fov>1.50098</horizontal_fov>
-          <lens>
-            <intrinsics>
-              <!-- fx = fy = width / ( 2 * tan (hfov / 2 ) ) -->
-              <fx>343.159</fx>
-              <fy>343.159</fy>
-              <!-- cx = ( width - 1 ) / 2 -->
-              <cx>319.5</cx>
-              <!-- cy = ( height - 1 ) / 2 -->
-              <cy>179.5</cy>
-              <s>0</s>
-            </intrinsics>
-          </lens>
-          <distortion>
-            <k1>0.0</k1>
-            <k2>0.0</k2>
-            <k3>0.0</k3>
-            <p1>0.0</p1>
-            <p2>0.0</p2>
-            <center>0.5 0.5</center>
-          </distortion>
-          <image>
-            <width>640</width>
-            <height>360</height>
-            <format>R8G8B8</format>
-          </image>
-          <clip>
-            <near>0.01</near>
-            <far>300</far>
-          </clip>
-          <depth_camera>
-            <clip>
-              <near>0.1</near>
-              <far>10</far>
-            </clip>
-          </depth_camera>
-          <noise>
-            <type>gaussian</type>
-            <mean>0</mean>
-            <stddev>0.007</stddev>
-          </noise>
-        </camera>
-      </sensor>
-    </gazebo>
+    <xacro:include filename="$(find lampo_description)/urdf/mm_arm.xacro" />
   </xacro:if>
 </robot>
