Commit message: okish

File: ros_ws/src/lampo_description/urdf/mm_arm.xacro (robot description, xacro)
@@ -16,5 +16,4 @@
   <xacro:arg name="safety_pos_margin" default="0.15"/>
   <xacro:arg name="safety_k_position" default="20"/>
-  <xacro:arg name="simulation_controllers" default="$(find lampo_description)/config/ur_controllers.yaml" />
   <xacro:arg name="ros_namespace" default="$(arg prefix)" />
   <!-- arm -->

File: ros_ws/src/lampo_description/urdf/mm_camera.xacro (robot description, xacro)
@@ -9,6 +9,6 @@
   </link>
   <joint name="$(arg prefix)cam_joint" type="fixed">
-    <origin xyz="0.0 0.0 0.1" rpy="0 0 0" />
-    <parent link="$(arg prefix)wrist_2_link" />
+    <origin xyz="0.0 -0.1 0.0" rpy="0 -1.57 1.57" />
+    <parent link="$(arg prefix)wrist_3_link" />
     <child link="$(arg prefix)cam_link" />
   </joint>

File: ros_ws/src/lampo_description/urdf/system.urdf.xacro (robot description, xacro)
@@ -3,4 +3,5 @@
   <xacro:arg name="omni" default="false" />
   <xacro:arg name="mm" default="false" />
+  <xacro:arg name="simulation_controllers" default="$(find lampo_description)/config/ur_controllers.yaml" />
   <xacro:if value="$(arg omni)">
     <xacro:include filename="$(find lampo_description)/urdf/sweepee/sweepee_omni.xacro" />
